Commit message: error fix

File: mycobot_ros/mycobot_description/urdf/mycobot_320_m5_2022/new_mycobot_pro_320moveit_m5_2022.urdf (robot description, URDF)
Before this commit: robot firefighter, 17 links, 16 joints
Links:
- added link closet; collision box size=1.040 0.4 0.0045; visual mesh filename=package://mycobot_description/urdf/mycobot_320_m5_2022/dres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
Joints:
- added joint base_to_closet: type fixed, parent base, child closet, origin xyz=-0.4 0 0.155 rpy=0 0 1.5708 
